Commit message: Fixed xacro issues with Baxter. Baxter now visualizes properly

File: baxter_common/baxter_description/urdf/left_end_effector.urdf (robot description, URDF)
Before this commit: robot left_end_effector, 1 links, 0 joints
Links:
- removed link l_gripper_l_finger
- added link l_side_l_finger, mass 0.02; collision box size=0.01 0.0135 0.1127; collision box size=0.01 0.05 0.017
- added link l_side_l_finger_tip, mass 0.01; collision box size=0.042 0.0065 0.037; visual mesh filename=package://rethink_ee_description/meshes/electric_gripper/fi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
- added link l_side_r_finger, mass 0.02; collision box size=0.01 0.0135 0.1127; collision box size=0.01 0.05 0.017
- added link l_side_r_finger_tip, mass 0.01; collision box size=0.042 0.0065 0.037; visual mesh filename=package://rethink_ee_description/meshes/electric_gripper/fi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
- added link left_gripper, mass 0.0001
- added link left_gripper_base, mass 0.3; collision cylinder length=0.1 radius=0.029; visual mesh filename=package://rethink_ee_description/meshes/electric_gripper/el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
Joints:
- added joint l_gripper_l_finger_joint: type prismatic, parent left_gripper_base, child l_gripper_l_finger, origin xyz=0.0 -0.0015 0.02 rpy=0 0 0, axis 0 1 0, limit lower=0.0 upper=0.020833 effort=20.0 velocity=5.0
- added joint l_gripper_r_finger_joint: type prismatic, parent left_gripper_base, child l_gripper_r_finger, origin xyz=0.0 0.0015 0.02 rpy=0 0 0, axis 0 1 0, limit lower=-0.020833 upper=0.0 effort=20.0 velocity=5.0, mimic joint=l_gripper_l_finger_joint multiplier=-1.0
- added joint l_side_l_finger_tip_joint: type fixed, parent l_side_l_finger, child l_side_l_finger_tip, origin xyz=0.0 0.01725 0.1127 rpy=0 0 0
- added joint l_side_r_finger_tip_joint: type fixed, parent l_side_r_finger, child l_side_r_finger_tip, origin xyz=0.0 -0.01725 0.1127 rpy=0 0 0
- added joint left_endpoint: type fixed, parent left_gripper_base, child left_gripper, origin xyz=0 0 0.02 rpy=0 0 0
- added joint left_gripper_base: type fixed, parent left_hand, child left_gripper_base, origin xyz=0 0 0.025 rpy=0 0 0

File: baxter_common/rethink_ee_description/urdf/electric_gripper/fingers/extended_narrow.xacro (robot description, xacro)
@@ -4,5 +4,5 @@
   <xacro:property name="finger_length" value="0.1127" scope="local"/>
   <xacro:property name="finger_width" value="0.01725" scope="local"/>
-  <xacro:property name="link_name" value="${gripper_side}_gripper" scope="local"/>
+  <xacro:property name="link_name" value="${gripper_side}_gripper_${finger_side}_finger" scope="local"/>
   <xacro:property name="collision_name" value="${link_name}_collision" scope="local"/>
   <xacro:property name="sensor_name" value="${link_name}_contact_sensor" scope="local"/>
@@ -50,7 +50,7 @@
           <collision>${collision_name}_collision</collision>
         </contact>
-        <plugin name="${gripper_side}_side_gripper_bumper" filename="libgazebo_ros_bumper.so">
+        <plugin name="${link_name}_bumper" filename="libgazebo_ros_bumper.so">
           <bumperTopicName>${gripper_side}_side_gripper_contact_sensor_state</bumperTopicName>
-          <frameName>${gripper_side}_side_gripper</frameName>
+          <frameName>${link_name}_frame</frameName>
         </plugin>
       </sensor>
