Commit message: Fixed fingers, added contact sensors to all fingers

File: baxter_common/baxter_description/urdf/left_end_effector.urdf.xacro (robot description, xacro)
@@ -3,9 +3,9 @@
   <xacro:include filename="$(find rethink_ee_description)/urdf/electric_gripper/rethink_electric_gripper.xacro" />
   <xacro:rethink_electric_gripper side="left"
-                                  l_finger="extended_narrow"
+                                  l_finger="standard_narrow"
                                   l_finger_slot="2"
                                   l_finger_tip="paddle_tip"
                                   l_finger_grasp="inner"
-                                  r_finger="extended_narrow"
+                                  r_finger="standard_narrow"
                                   r_finger_slot="2"
                                   r_finger_tip="paddle_tip"

File: baxter_common/baxter_description/urdf/right_end_effector.urdf.xacro (robot description, xacro)
@@ -3,11 +3,11 @@
   <xacro:include filename="$(find rethink_ee_description)/urdf/electric_gripper/rethink_electric_gripper.xacro" />
   <xacro:rethink_electric_gripper side="right"
-                                  l_finger="extended_narrow"
+                                  l_finger="standard_narrow"
                                   l_finger_slot="2"
-                                  l_finger_tip="half_round_tip"
+                                  l_finger_tip="paddle_tip"
                                   l_finger_grasp="inner"
-                                  r_finger="extended_narrow"
+                                  r_finger="standard_narrow"
                                   r_finger_slot="2"
-                                  r_finger_tip="half_round_tip"
+                                  r_finger_tip="paddle_tip"
                                   r_finger_grasp="inner"/>
 </robot>

File: baxter_common/rethink_ee_description/urdf/electric_gripper/fingers/extended_wide.xacro (robot description, xacro)
@@ -2,7 +2,10 @@
 <robot xmlns:xacro="http://www.ros.org/wiki/xacro" name="wide_extended">
   <xacro:macro name="finger_xacro" params="gripper_side finger_side reflect finger_tip finger_grasp">
-    <xacro:property name="finger_length" value="0.1127" scope="global"/>
-    <xacro:property name="finger_width" value="0.05503" scope="local"/>
-    <link name="${gripper_side}_gripper_${finger_side}_finger">
+  <xacro:property name="finger_length" value="0.1127" scope="global"/>
+  <xacro:property name="finger_width" value="0.05503" scope="local"/>
+  <xacro:property name="link_name" value="${gripper_side}_gripper_${finger_side}_finger" scope="local"/>
+  <xacro:property name="collision_name" value="${link_name}_collision" scope="local"/>
+  <xacro:property name="sensor_name" value="${link_name}_contact_sensor" scope="local"/>
+    <link name="${link_name}">
       <visual>
         <origin rpy="0 0 ${-pi/2*(reflect+1)}" xyz="0 0 0"/>
@@ -11,8 +14,8 @@
         </geometry>
       </visual>
-     <xacro:property name="finger_box_height" value="0.01" scope="local"/>
-     <xacro:property name="finger_box_width" value="0.0135" scope="local"/>
-     <xacro:property name="finger_box_length" value="0.0615" scope="local"/>
-     <collision>
+      <xacro:property name="finger_box_height" value="0.01" scope="local"/>
+      <xacro:property name="finger_box_width" value="0.0135" scope="local"/>
+      <xacro:property name="finger_box_length" value="0.0615" scope="local"/>
+      <collision name="${collision_name}">
         <origin rpy="0 0 ${-pi/2*(reflect+1)}" xyz="0 ${finger_width*reflect} ${finger_box_length}"/>
         <geometry>
@@ -35,5 +38,5 @@
       </inertial>
     </link>
-    <gazebo reference="${gripper_side}_gripper_${finger_side}_finger">
+    <gazebo reference="${link_name}">
       <mu1>1000</mu1>
       <mu2>1000</mu2>
@@ -41,4 +44,15 @@
       <kp>1e5</kp>
       <kd>1.0</kd>
+      <sensor name="${sensor_name}" type="contact">
+        <always_on>true</always_on>
+        <update_rate>30</update_rate>
+        <contact>
+          <collision>${collision_name}_collision</collision>
+        </contact>
+        <plugin name="${link_name}_bumper" filename="libgazebo_ros_bumper.so">
+          <bumperTopicName>${gripper_side}_side_gripper_contact_sensor_state</bumperTopicName>
+          <frameName>${link_name}_frame</frameName>
+        </plugin>
+      </sensor>
     </gazebo>
    <xacro:property name="none" value="[none, false, null, empty]" scope="local"/>
@@ -47,5 +61,5 @@
    </xacro:if>
    <xacro:include filename="$(find rethink_ee_description)/urdf/electric_gripper/fingers/${finger_tip}.xacro" />
-   <xacro:finger_tip_xacro parent_link="${gripper_side}_gripper_${finger_side}_finger" reflect="${reflect}" grasp="${finger_grasp}">
+   <xacro:finger_tip_xacro parent_link="${link_name}" reflect="${reflect}" grasp="${finger_grasp}">
        <origin rpy="0 0 0" xyz="0.0 ${reflect*finger_width} ${finger_length}"/>
    </xacro:finger_tip_xacro>

File: baxter_common/rethink_ee_description/urdf/electric_gripper/fingers/standard_narrow.xacro (robot description, xacro)
@@ -4,5 +4,8 @@
   <xacro:property name="finger_length" value="0.075" scope="global"/>
   <xacro:property name="finger_width" value="0.01725" scope="local"/>
-    <link name="${gripper_side}_gripper_${finger_side}_finger">
+  <xacro:property name="link_name" value="${gripper_side}_gripper_${finger_side}_finger" scope="local"/>
+  <xacro:property name="collision_name" value="${link_name}_collision" scope="local"/>
+  <xacro:property name="sensor_name" value="${link_name}_contact_sensor" scope="local"/>
+    <link name="${link_name}">
       <visual>
         <origin rpy="0 0 ${-pi/2*(reflect+1)}" xyz="0 0 0"/>
@@ -14,5 +17,5 @@
       <xacro:property name="finger_box_width" value="0.0135" scope="local"/>
       <xacro:property name="finger_box_length" value="0.04" scope="local"/>
-      <collision>
+      <collision name="${collision_name}">
         <origin rpy="0 0 ${-pi/2*(reflect+1)}" xyz="0 ${finger_width*reflect} ${finger_box_length}"/>
         <geometry>
@@ -35,5 +38,5 @@
       </inertial>
     </link>
-    <gazebo reference="${gripper_side}_gripper_${finger_side}_finger">
+    <gazebo reference="${link_name}">
       <mu1>1000</mu1>
       <mu2>1000</mu2>
@@ -41,4 +44,15 @@
       <kp>1e5</kp>
       <kd>1.0</kd>
+      <sensor name="${sensor_name}" type="contact">
+        <always_on>true</always_on>
+        <update_rate>30</update_rate>
+        <contact>
+          <collision>${collision_name}_collision</collision>
+        </contact>
+        <plugin name="${link_name}_bumper" filename="libgazebo_ros_bumper.so">
+          <bumperTopicName>${gripper_side}_side_gripper_contact_sensor_state</bumperTopicName>
+          <frameName>${link_name}_frame</frameName>
+        </plugin>
+      </sensor>
     </gazebo>
    <xacro:property name="none" value="[none, false, null, empty]" scope="local"/>
@@ -47,5 +61,5 @@
    </xacro:if>
    <xacro:include filename="$(find rethink_ee_description)/urdf/electric_gripper/fingers/${finger_tip}.xacro" />
-   <xacro:finger_tip_xacro parent_link="${gripper_side}_gripper_${finger_side}_finger" reflect="${reflect}" grasp="${finger_grasp}">
+   <xacro:finger_tip_xacro parent_link="${link_name}" reflect="${reflect}" grasp="${finger_grasp}">
        <origin rpy="0 0 0" xyz="0.0 ${reflect*finger_width} ${finger_length}"/>
    </xacro:finger_tip_xacro>

File: baxter_common/rethink_ee_description/urdf/electric_gripper/fingers/standard_wide.xacro (robot description, xacro)
@@ -4,5 +4,8 @@
   <xacro:property name="finger_length" value="0.075" scope="global"/>
   <xacro:property name="finger_width" value="0.05503" scope="local"/>
-    <link name="${gripper_side}_gripper_${finger_side}_finger">
+  <xacro:property name="link_name" value="${gripper_side}_gripper_${finger_side}_finger" scope="local"/>
+  <xacro:property name="collision_name" value="${link_name}_collision" scope="local"/>
+  <xacro:property name="sensor_name" value="${link_name}_contact_sensor" scope="local"/>
+    <link name="${link_name}">
       <visual>
         <origin rpy="0 0 ${-pi/2*(reflect+1)}" xyz="0 0 0"/>
@@ -14,5 +17,5 @@
       <xacro:property name="finger_box_width" value="0.0135" scope="local"/>
       <xacro:property name="finger_box_length" value="0.04" scope="local"/>
-      <collision>
+      <collision name="${collision_name}">
         <origin rpy="0 0 ${-pi/2*(reflect+1)}" xyz="0 ${finger_width*reflect} ${finger_box_length}"/>
         <geometry>
@@ -35,5 +38,5 @@
       </inertial>
     </link>
-    <gazebo reference="${gripper_side}_gripper_${finger_side}_finger">
+    <gazebo reference="${link_name}">
       <mu1>1000</mu1>
       <mu2>1000</mu2>
@@ -41,4 +44,15 @@
       <kp>1e5</kp>
       <kd>1.0</kd>
+      <sensor name="${sensor_name}" type="contact">
+        <always_on>true</always_on>
+        <update_rate>30</update_rate>
+        <contact>
+          <collision>${collision_name}_collision</collision>
+        </contact>
+        <plugin name="${link_name}_bumper" filename="libgazebo_ros_bumper.so">
+          <bumperTopicName>${gripper_side}_side_gripper_contact_sensor_state</bumperTopicName>
+          <frameName>${link_name}_frame</frameName>
+        </plugin>
+      </sensor>
     </gazebo>
    <xacro:property name="none" value="[none, false, null, empty]" scope="local"/>
@@ -47,5 +61,5 @@
    </xacro:if>
    <xacro:include filename="$(find rethink_ee_description)/urdf/electric_gripper/fingers/${finger_tip}.xacro" />
-   <xacro:finger_tip_xacro parent_link="${gripper_side}_gripper_${finger_side}_finger" reflect="${reflect}" grasp="${finger_grasp}">
+   <xacro:finger_tip_xacro parent_link="${link_name}" reflect="${reflect}" grasp="${finger_grasp}">
        <origin rpy="0 0 0" xyz="0.0 ${reflect*finger_width} ${finger_length}"/>
    </xacro:finger_tip_xacro>
